Commit message: wip

File: example_1/description/ros2_control/rrbot.ros2_control.xacro (robot description, xacro)
@@ -1,6 +1,10 @@
 <?xml version="1.0"?>
 <robot xmlns:xacro="http://www.ros.org/wiki/xacro">
-  <xacro:macro name="rrbot_ros2_control" params="name prefix">
-    <ros2_control name="${name}" type="system">
+  <xacro:macro
+      name="rrbot_ros2_control"
+      params="name prefix">
+    <ros2_control
+        name="${name}"
+        type="sensor">
       <hardware>
         <plugin>ros2_control_demo_example_1/RRBotSystemPositionOnlyHardware</plugin>
@@ -9,18 +13,12 @@
         <param name="example_param_hw_slowdown">100</param>
       </hardware>
-      <joint name="${prefix}joint1">
-        <command_interface name="position">
-          <param name="min">-1</param>
-          <param name="max">1</param>
-        </command_interface>
-        <state_interface name="position"/>
-      </joint>
-      <joint name="${prefix}joint2">
-        <command_interface name="position">
-          <param name="min">-1</param>
-          <param name="max">1</param>
-        </command_interface>
-        <state_interface name="position"/>
-      </joint>
+      <sensor name="${prefix}image_sensor">
+        <state_interface name="height" />
+        <state_interface name="width" />
+        <state_interface name="encoding" />
+        <state_interface name="is_bigendian" />
+        <state_interface name="step" />
+        <state_interface name="data" />
+      </sensor>
     </ros2_control>
   </xacro:macro>
